File: pcb/wombat.sch (KiCad schematic (older format))
At the start: 0 parts

Commit message: schematic finished, parts specced for gps
Parts:
- added ANT1: SL1200, symbol SL1200
- added BATT1: COINCELL, symbol COINCELL
- added C1, C11, C3: 100n, SM0402, symbol C
- added C10, C20, C21, C22, C23, C42, C47: 100n, symbol C
- added C12, C14, C15, C18: 1µ, symbol C
- added C13, C24, C4: 4µ7, symbol C
- added C16, C17, C25, C30, C45: 10n, symbol C
- added C19, C38: 3p3, symbol C
- added C2: 1µ, SM0402, symbol C
- added C26: 680p, symbol C
- added C27: 12n, symbol C
- added C28: 270p, symbol C
- added C29: 22n, symbol C
- added C31: 470n, symbol C
- added C32: 8p2, symbol C
- added C33, C34, C35: 2µ2, symbol C
- added C36, C41: SPEC ME, symbol C
- added C37, C40: 18p, symbol C
- added C39: 470p, symbol C
- added C43, C44: 5p1, symbol C
- added C46, C7, C8, C9: 10µ, symbol C
- added C5: 15p, SM0402, symbol C
- added C6: 6p8, SM0402, symbol C
- added D1, D2: USBLC6-2, symbol USBLC6-2
- added D3, D4, D5: LED, symbol LED
- added IC1: MCP73831, symbol MCP73831
- added IC2: TPS61201, symbol TPS61201
- added IC3: 24AA32A, MSOP8, symbol 24AA32A
- added IC4: TPS76933DBVT, symbol TPS76933DBVT
- added IC5: TC1016, symbol TC1016
- added IC6: TMP102, symbol TMP102
- added IC7: ADF7012, symbol ADF7012
- added IC8: STM32F405RGT6, symbol STM32F405RGT6
- added L1: 2µ2, symbol INDUCTOR
- added L2: 22n, SM0402, symbol INDUCTOR
- added L3: 6n8, SM0402, symbol INDUCTOR
- added L4, L6, L7: 22n, symbol INDUCTOR
- added L5: 27n, symbol INDUCTOR
- added L8: 6n2, symbol INDUCTOR
- added P1: LiPo, symbol CONN_2
- added P10: CUTDOWN, symbol CONN_2
- added P11, P12, P13, P14, P15, P16, P17, P18, P19, P2, P20, P21, P22, P23, P25, P4, P5, P6, P7, P8, P9: TST, symbol TST
- added P24: CONN_6, symbol CONN_6
- added P3: BATT, symbol CONN_2
- added Q1: MOSFET_N, symbol MOSFET_N
- added Q2, Q3: BC817, symbol NPN
- added R1: 12R, SM0402, symbol R
- added R10, R7: 4k7, symbol R
- added R11: 15k, symbol R
- added R12: 47k, symbol R
- added R13: 36k, symbol R
- added R14: 22k, symbol R
- added R15, R31, R8: 10k, symbol R
- added R16, R20, R22, R23, R26, R28, R29, R30, R32: 1k, symbol R
- added R17: 1k5, symbol R
- added R18: 3k3, symbol R
- added R19: 910, symbol R
- added R2: 10k, SM0402, symbol R
- added R21: 3k6, symbol R
- added R24, R25, R27: 330, symbol R
- added R3, R33, R34, R6: 22, SM0402, symbol R
- added R4: 2k, symbol R
- added R5: 8k2, SM0402, symbol R
- added R9: 100R, symbol R
- added SJ1, SJ2: SJ, symbol SJ
- added SMA1: SMA_JACK, symbol SMA_JACK
- added SW1, SW2: SW_PUSH, symbol SW_PUSH
- added U1: NEO6Q, NEO6Q, symbol NEO6Q
- added U2: ALM-1712, ALM-1712, symbol ALM-1712
- added USB1, USB2: MICROUSB, symbol MICROUSB
- added X1: 4.9152MHz, symbol CRYSTAL
- added X2: 8MHz, symbol CRYSTAL
Connections:
- net labels added: 2V7, 3V3, ADF_CE, ADF_CLK, ADF_CLKOUT, ADF_DATA, ADF_LE, ADF_MUXOUT, ADF_TXCLK, ADF_TXDATA, BOOT0, CHG_STAT, CUTDOWN1, GND, GPS_DM, GPS_DP, GPS_RX, GPS_TX, NRST, STM_DM, STM_DP, STM_USB_DISC, STM_USB_V, TMP_SCL, TMP_SDA, USART1_RX, USART1_TX, VBATT, VBUS, VBUS_3V3, VIN
- wire segments 0 -> 485
- no-connect marks 0 -> 46
Other:
- note added: "Backup\nBattery"
- note added: "Boot Config:\nSelf Powered"
- note added: "CP\nFilter"
- note added: "CUTDOWN"
- note added: "Config EEPROM"
- note added: "ESD Protection"
- note added: "FTDI HEADER"
- note added: "GPS"
- note added: "GPS USB VREG"
- note added: "GPS\nUSB"
- note added: "LNA"
- note added: "LNA 2v7 VREG"
- note added: "LiPo Charging"
- note added: "MAIN 3v3 SMPS"
- note added: "Output\nFilter"
- note added: "POWER MANAGEMENT"
- note added: "RADIO"
- note added: "RESET &\nBOOTLOAD"
- note added: "SJs for\nSTM32F1"
- note added: "SPI1"
- note added: "SPI2"
- note added: "STM USB Disconnect"
- note added: "STM USB\nDetect"
- note added: "STM32"
- note added: "STM\nUSB"
- note added: "TEMPERATURE\nSENSOR"
- note added: "TIM2_CH3"
- note added: "USART1"
- note added: "USART2"
- note added: "USB"

Commit message: spec cutdown parts
Parts:
- P10: footprint (none) -> BLOCK-3.5-2; Farnell (none) -> 1098611
- Q1: footprint (none) -> SOT-23; Farnell (none) -> 1758067
- R15: footprint (none) -> SM0402; Farnell (none) -> 1738864
- R9: footprint (none) -> SM0402; Farnell (none) -> 1738837
Changed lines of the file:
@@
-EESchema Schematic File Version 2  date Sun 19 Feb 2012 22:56:49 GMT
+EESchema Schematic File Version 2  date Sun 19 Feb 2012 23:03:55 GMT
 LIBS:power
 LIBS:device
@@
 F 0 "R9" V 2780 3250 50  0000 C CNN
 F 1 "100R" V 2700 3250 50  0000 C CNN
+F 2 "SM0402" H 2700 3250 60  0001 C CNN
+F 4 "1738837" H 2700 3250 60  0001 C CNN "Farnell"
 	1    2700 3250
 	0    1    1    0
@@
 F 0 "R15" V 2830 3500 50  0000 C CNN
 F 1 "10k" V 2750 3500 50  0000 C CNN
+F 2 "SM0402" H 2750 3500 60  0001 C CNN
+F 4 "1738864" H 2750 3500 60  0001 C CNN "Farnell"
 	1    2750 3500
 	0    1    1    0
@@
 F 0 "P10" V 3850 3250 40  0000 C CNN
 F 1 "CUTDOWN" V 3950 3250 40  0000 C CNN
+F 2 "BLOCK-3.5-2" H 3900 3250 60  0001 C CNN
+F 4 "1098611" H 3900 3250 60  0001 C CNN "Farnell"
 	1    3900 3250
 	1    0    0    -1
@@
 F 0 "Q1" H 3260 3420 60  0000 R CNN
 F 1 "MOSFET_N" H 3260 3100 60  0000 R CNN
+F 2 "SOT-23" H 3250 3250 60  0001 C CNN
+F 4 "1758067" H 3250 3250 60  0001 C CNN "Farnell"
 	1    3250 3250
 	1    0    0    -1

Commit message: spec temp sensor parts
Parts:
- C16: footprint (none) -> SM0402; Farnell (none) -> 1740589
- IC6: footprint (none) -> SOT563; Farnell (none) -> 1652477
- R10, R7: footprint (none) -> SM0402; Farnell (none) -> 1738858
Changed lines of the file:
@@
-EESchema Schematic File Version 2  date Sun 19 Feb 2012 23:03:55 GMT
+EESchema Schematic File Version 2  date Sun 19 Feb 2012 23:06:54 GMT
 LIBS:power
 LIBS:device
@@
 F 0 "R7" V 4730 3100 50  0000 C CNN
 F 1 "4k7" V 4650 3100 50  0000 C CNN
+F 2 "SM0402" H 4650 3100 60  0001 C CNN
+F 4 "1738858" H 4650 3100 60  0001 C CNN "Farnell"
 	1    4650 3100
 	0    1    1    0
@@
 F 0 "R10" V 4780 3250 50  0000 C CNN
 F 1 "4k7" V 4700 3250 50  0000 C CNN
+F 2 "SM0402" H 4700 3250 60  0001 C CNN
+F 4 "1738858" H 4700 3250 60  0001 C CNN "Farnell"
 	1    4700 3250
 	0    1    1    0
@@
 F 0 "C16" H 5150 3550 50  0000 L CNN
 F 1 "10n" H 5150 3350 50  0000 L CNN
+F 2 "SM0402" H 5100 3450 60  0001 C CNN
+F 4 "1740589" H 5100 3450 60  0001 C CNN "Farnell"
 	1    5100 3450
 	1    0    0    -1
@@
 F 0 "IC6" H 5350 3650 60  0000 C CNN
 F 1 "TMP102" H 5450 3250 60  0000 C CNN
+F 2 "SOT563" H 5550 3450 60  0001 C CNN
+F 4 "1652477" H 5550 3450 60  0001 C CNN "Farnell"
 	1    5550 3450
 	0    1    1    0

Commit message: spec all stm parts
Parts:
- removed C36, C41: SPEC ME, symbol C
- removed X2: 8MHz, symbol CRYSTAL
- added X2: 8MHz, RESONATOR, symbol RESONATOR
- C17: footprint (none) -> SM0402; Farnell (none) -> 1740589
- C18: footprint (none) -> SM0402; Farnell (none) -> 1288253
- C20, C21, C22, C23: footprint (none) -> SM0402; Farnell (none) -> 1828862
- C24: footprint (none) -> SM0603; Farnell (none) -> 1833803
- C33, C34: footprint (none) -> SM0603; Farnell (none) -> 1833808
- D3, D4, D5: footprint (none) -> SM0603; Farnell (none) -> 8529850
- IC8: footprint (none) -> LQFP64; Farnell (none) -> 2064363
- R24, R25, R27: footprint (none) -> SM0402; Farnell (none) -> 1738843
- SJ1, SJ2: footprint (none) -> SJ
Connections:
- wire segments 485 -> 481

Commit message: spec ftdi parts
Parts:
- C47: footprint (none) -> SM0402; Farnell (none) -> 1828862
- P24: footprint (none) -> HEADER_SMD_6WAY; Farnell (none) -> 9689508
Changed lines of the file:
@@
-EESchema Schematic File Version 2  date Sun 19 Feb 2012 23:33:20 GMT
+EESchema Schematic File Version 2  date Sun 19 Feb 2012 23:36:19 GMT
 LIBS:power
 LIBS:device
@@
 F 0 "C47" H 6200 7750 50  0000 L CNN
 F 1 "100n" H 6200 7550 50  0000 L CNN
+F 2 "SM0402" H 6150 7650 60  0001 C CNN
+F 4 "1828862" H 6150 7650 60  0001 C CNN "Farnell"
 	1    6150 7650
 	0    -1   -1   0
@@
 F 0 "P24" V 6750 7400 60  0000 C CNN
 F 1 "CONN_6" V 6850 7400 60  0000 C CNN
+F 2 "HEADER_SMD_6WAY" H 6800 7400 60  0001 C CNN
+F 4 "9689508" H 6800 7400 60  0001 C CNN "Farnell"
 	1    6800 7400
 	1    0    0    -1

Commit message: spec reset and bootload parts
Parts:
- R31: footprint (none) -> SM0402; Farnell (none) -> 1738864
- SW1, SW2: footprint (none) -> SMDSWITCH; Farnell (none) -> 1607971
Changed lines of the file:
@@
-EESchema Schematic File Version 2  date Sun 19 Feb 2012 23:36:19 GMT
+EESchema Schematic File Version 2  date Sun 19 Feb 2012 23:39:04 GMT
 LIBS:power
 LIBS:device
@@
 F 0 "R31" V 5730 6600 50  0000 C CNN
 F 1 "10k" V 5650 6600 50  0000 C CNN
+F 2 "SM0402" H 5650 6600 60  0001 C CNN
+F 4 "1738864" H 5650 6600 60  0001 C CNN "Farnell"
 	1    5650 6600
 	0    1    1    0
@@
 F 0 "SW2" H 5850 6510 50  0000 C CNN
 F 1 "SW_PUSH" H 5700 6320 50  0000 C CNN
+F 2 "SMDSWITCH" H 5700 6400 60  0001 C CNN
+F 4 "1607971" H 5700 6400 60  0001 C CNN "Farnell"
 	1    5700 6400
 	1    0    0    -1
@@
 F 0 "SW1" H 5850 6260 50  0000 C CNN
 F 1 "SW_PUSH" H 5700 6070 50  0000 C CNN
+F 2 "SMDSWITCH" H 5700 6150 60  0001 C CNN
+F 4 "1607971" H 5700 6150 60  0001 C CNN "Farnell"
 	1    5700 6150
 	1    0    0    -1

Commit message: stm32 to resonator and cutdown updated
Parts:
- added C?: 100n, SM0402, symbol C
- added C?: 4700µ, RADIAL-5, symbol CP1
- added L?: FB, SM0603, symbol INDUCTOR
- added R? (x2): 10k, SM0402, symbol R
- added R?: 100R, SM0402, symbol R
- C25, C30, C45: footprint (none) -> SM0402; Farnell (none) -> 1740589
- C26: footprint (none) -> SM0402; Farnell (none) -> 1865453
- C27: footprint (none) -> SM0402; Farnell (none) -> 1865461
- C28: footprint (none) -> SM0402; Farnell (none) -> 1414585
- C29: footprint (none) -> SM0402; Farnell (none) -> 1414583
- C31: footprint (none) -> SM0402; Farnell (none) -> 1414593
- C35: footprint (none) -> SM0603; Farnell (none) -> 1833808
- C37, C40: footprint (none) -> SM0402; Farnell (none) -> 1740572
- C42: footprint (none) -> SM0402; Farnell (none) -> 1828862
- L7: footprint (none) -> SM0402; Farnell (none) -> 1669580
- P10: value CUTDOWN -> PYRO
- R18, R21: footprint (none) -> SM0402; Farnell (none) -> 1738856
- R19: footprint (none) -> SM0402; Farnell (none) -> 1458832
- R20, R22, R23, R26, R28, R29, R30, R32: footprint (none) -> SM0402; Farnell (none) -> 1738850
- X1: footprint (none) -> HC49; Farnell (none) -> 1640864
Connections:
- net labels added: PYRO_FIRE, PYRO_TEST
- net labels removed: CUTDOWN1
- wire segments 481 -> 608
- no-connect marks 46 -> 45
Other:
- note added: "Capacitor current limiting\n (may be 0R)"
- note added: "Use 2R 8W\n inline\n ballast"
- moved on the sheet: C17, C18, R15, R9

Commit message: update load caps on adf crystal 18->26pF (so that total C_L=18pF)
Parts:
- C37, C40: value 18p -> 26p; Farnell 1740572 -> 1414584
Changed lines of the file:
@@
-EESchema Schematic File Version 2  date Wed 22 Feb 2012 04:05:50 GMT
+EESchema Schematic File Version 2  date Wed 22 Feb 2012 04:14:24 GMT
 LIBS:power
 LIBS:device
@@
 P 6550 6150
 F 0 "C40" H 6600 6250 50  0000 L CNN
-F 1 "18p" H 6600 6050 50  0000 L CNN
+F 1 "26p" H 6600 6050 50  0000 L CNN
 F 2 "SM0402" H 6550 6150 60  0001 C CNN
-F 4 "1740572" H 6550 6150 60  0001 C CNN "Farnell"
+F 4 "1414584" H 6550 6150 60  0001 C CNN "Farnell"
 	1    6550 6150
 	0    -1   -1   0
@@
 P 6550 5550
 F 0 "C37" H 6600 5650 50  0000 L CNN
-F 1 "18p" H 6600 5450 50  0000 L CNN
+F 1 "26p" H 6600 5450 50  0000 L CNN
 F 2 "SM0402" H 6550 5550 60  0001 C CNN
-F 4 "1740572" H 6550 5550 60  0001 C CNN "Farnell"
+F 4 "1414584" H 6550 5550 60  0001 C CNN "Farnell"
 	1    6550 5550
 	0    -1   -1   0
