File: pcb/wombat.sch (KiCad schematic (older format))
At the start: 147 parts, among them IC1 MCP73831, IC2 TPS61201, IC3 24AA32A, IC4 TPS76933DBVT, IC5 TC1016, IC6 TMP102, IC7 ADF7012, IC8 STM32F405RGT6, P1 LiPo, P10 PYRO, P11 TST, P12 TST, P13 TST, P14 TST, P15 TST, P16 TST, P17 TST, P18 TST, P19 TST, P2 TST, P20 TST, P21 TST, P22 TST, P23 TST, P24 CONN_6, P25 TST, P3 BATT, P4 TST, P5 TST, P6 TST, P7 TST, P8 TST, P9 TST, Q1 MOSFET_N, Q2 BC817, Q3 BC817, SW1 SW_PUSH, SW2 SW_PUSH, U1 NEO6Q, U2 ALM-1712, X1 4.9152MHz, X2 8MHz

Commit message: radio section all specced
Parts:
- added D6: LED, SM0603, symbol LED
- added R32: 330, SM0402, symbol R
- C21: renamed from C19; footprint (none) -> SM0402; Farnell (none) -> 1702752
- C34: renamed from C32; footprint (none) -> SM0402; Farnell (none) -> 7568118
- C39: renamed from C38; footprint (none) -> SM0402; Farnell (none) -> 1702752
- C40: renamed from C39; footprint (none) -> SM0402; Farnell (none) -> 1535556
- C43, C44: footprint (none) -> SM0402; Farnell (none) -> 1885321
- C46: footprint (none) -> SM0603; Farnell (none) -> 1735528
- IC7: footprint (none) -> TSSOP24; Farnell (none) -> 1346367
- L5: renamed from L4; footprint (none) -> SM0402; Farnell (none) -> 1669580
- L6: renamed from L5; footprint (none) -> SM0402; Farnell (none) -> 1265429
- L7: renamed from L6; footprint (none) -> SM0402; Farnell (none) -> 1669580
- L9: renamed from L8; footprint (none) -> SM0402; Farnell (none) -> 1265407
- SMA1: footprint (none) -> SMA_JACK_END_LAUNCH; Farnell (none) -> 1342651
- gave numbers to parts that had none: 6
- renumbered C16 to C18, C17 to C19, C18 to C20, C20 to C22, C21 to C23, C22 to C24, C23 to C25, C24 to C26, C25 to C27, C26 to C28, C27 to C29, C28 to C30, C29 to C31, C30 to C32, C31 to C33, C33 to C35, C34 to C36, C35 to C37, C37 to C38, C40 to C41, L7 to L8, P11 to P10, P12 to P11, P13 to P12, P10 to P13, R8 to R10, R10 to R12, R11 to R13, R15 to R14, R12 to R16, R13 to R17, R14 to R18, R16 to R19, R17 to R20, R18 to R21, R19 to R22, R20 to R23, R21 to R24, R22 to R25, R23 to R26, R24 to R27, R25 to R28, R26 to R29, R27 to R30, R28 to R31, R29 to R33, R30 to R34, R31 to R35, R32 to R36, R33 to R37, R34 to R38, R7 to R8, X2 to X1, X1 to X2
Connections:
- wire segments 608 -> 611
- no-connect marks 45 -> 44

Commit message: spec all power parts
Parts:
- added C12: 4µ7, SM0603, symbol C
- added C3: 10µ, SM0603, symbol C
- added R?: 100k, SM0402, symbol R
- added R?: 1M1, SM0402, symbol R
- BATT1: footprint (none) -> 2032HOLDER; Farnell (none) -> 1704232
- C10: renamed from C9; footprint (none) -> SM0603; Farnell (none) -> 1735528
- C11: renamed from C10; footprint (none) -> SM0402; Farnell (none) -> 1828862
- C14: renamed from C12; footprint (none) -> SM0402; Farnell (none) -> 1288253
- C15: renamed from C13; footprint (none) -> SM0603; Farnell (none) -> 1833803
- C16: renamed from C14; footprint (none) -> SM0402; Farnell (none) -> 1288253
- C17: renamed from C15; footprint (none) -> SM0402; Farnell (none) -> 1288253
- C5: renamed from C4; footprint (none) -> SM0603; Farnell (none) -> 1833803
- C8: renamed from C7; footprint (none) -> SM0603; Farnell (none) -> 1735528
- C9: renamed from C8; footprint (none) -> SM0603; Farnell (none) -> 1735528
- D1, D2: footprint (none) -> SOT-23; Farnell (none) -> 1857788
- IC1: footprint (none) -> SOT-23-5; Farnell (none) -> 1332158
- IC2: footprint (none) -> TPS61201; Farnell (none) -> 1564952
- IC4: footprint (none) -> SOT-23-5; Farnell (none) -> 8461538
- IC5: footprint (none) -> SOT-23-5; Farnell (none) -> 1825051
- L1: footprint (none) -> SM0805; Farnell (none) -> 1265551
- P1: footprint (none) -> JST-2mm-2; Farnell (none) -> 9492615
- P13: footprint BLOCK-3.5-2 -> BLOCK-3.5mm-2
- P3: footprint (none) -> BLOCK-3.5mm-2; Farnell (none) -> 1098611
- Q2, Q3: footprint (none) -> SOT-23-3; Farnell (none) -> 1081223
- R10: footprint (none) -> SM0402; Farnell (none) -> 1738864
- R13: footprint (none) -> SM0402; Farnell (none) -> 2059240
- R16: footprint (none) -> SM0402; Farnell (none) -> 2059246
- R17: footprint (none) -> SM0402; Farnell (none) -> 1358084
- R18: footprint (none) -> SM0402; Farnell (none) -> 2059243
- R19: footprint (none) -> SM0402; Farnell (none) -> 1738850
- R20: footprint (none) -> SM0402; Farnell (none) -> 2059227
- R4: footprint (none) -> SM0402; Farnell (none) -> 1358050
- USB1, USB2: footprint (none) -> MICROUSB; Farnell (none) -> 1521869
- renumbered C11 to C13, C16 to C18, C17 to C19, C18 to C20, C19 to C21, C20 to C22, C21 to C23, C22 to C24, C23 to C25, C24 to C26, C25 to C27, C26 to C28, C27 to C29, C28 to C30, C29 to C31, C30 to C32, C31 to C33, C32 to C34, C33 to C35, C34 to C36, C35 to C37, C36 to C38, C37 to C39, C3 to C4, C38 to C40, C39 to C41, C40 to C42, C41 to C43, C42 to C44, C43 to C45, C44 to C46, C45 to C47, C46 to C48, C47 to C49, C5 to C6, C6 to C7
Connections:
- wire segments 611 -> 520

Commit message: reannotate
Parts:
- gave numbers to parts that had none: 2
- renumbered C12 to C11, C11 to C12, R8 to R10, R9 to R11, R10 to R12, R11 to R13, R12 to R14, R13 to R15, R14 to R16, R15 to R17, R16 to R18, R17 to R19, R18 to R20, R19 to R21, R20 to R22, R21 to R23, R22 to R24, R23 to R25, R24 to R26, R25 to R27, R26 to R28, R27 to R29, R28 to R30, R29 to R31, R30 to R32, R31 to R33, R32 to R34, R33 to R35, R34 to R36, R35 to R37, R36 to R38, R37 to R39, R38 to R40, R7 to R9

Commit message: fix incorrect farnell code for 3k6 resistor
Parts:
- ANT1: footprint (none) -> SL1200
- R26: Farnell 1738856 -> 1358057
Changed lines of the file:
@@
-EESchema Schematic File Version 2  date Wed 22 Feb 2012 05:33:44 GMT
+EESchema Schematic File Version 2  date Wed 22 Feb 2012 05:42:40 GMT
 LIBS:power
 LIBS:device
@@
 F 1 "3k6" V 9200 5150 50  0000 C CNN
 F 2 "SM0402" H 9200 5150 60  0001 C CNN
-F 4 "1738856" H 9200 5150 60  0001 C CNN "Farnell"
+F 4 "1358057" H 9200 5150 60  0001 C CNN "Farnell"
 	1    9200 5150
 	0    1    1    0
@@
 F 0 "ANT1" H 750 1910 60  0000 C CNN
 F 1 "SL1200" H 750 1990 60  0000 C CNN
+F 2 "SL1200" H 750 1650 60  0001 C CNN
 	1    750  1650
 	1    0    0    -1
