File: pcb/wombat.sch (KiCad schematic (older format))
At the start: 153 parts, among them IC1 MCP73831, IC2 TPS61201, IC3 24AA32A, IC4 TPS76933DBVT, IC5 TC1016, IC6 TMP102, IC7 ADF7012, IC8 STM32F405RGT6, P1 LiPo, P10 TST, P11 TST, P12 TST, P13 PYRO, P14 TST, P15 TST, P16 TST, P17 TST, P18 TST, P19 TST, P2 TST, P20 TST, P21 TST, P22 TST, P23 TST, P24 CONN_6, P25 TST, P3 BATT, P4 TST, P5 TST, P6 TST, P7 TST, P8 TST, P9 TST, Q1 MOSFET_N, Q2 BC817, Q3 BC817, SW1 SW_PUSH, SW2 SW_PUSH, U1 NEO6Q, U2 ALM-1712, X1 8MHz, X2 4.9152MHz

Commit message: tidy up sch - remove silly d+ pullup, connect boot0 button to a gpio, add jtag header
Parts:
- removed Q2, Q3: BC817, SOT-23-3, symbol NPN
- removed R12: 10k, SM0402, symbol R
- removed R18: 47k, SM0402, symbol R
- removed R19: 36k, SM0402, symbol R
- removed R21: 1k, SM0402, symbol R
- added P26: CONN_10X2, HEADER_SMD_2X10WAY, symbol CONN_10X2
- added R41: 10k, SM0402, symbol R
- added R42: 1k, SM0402, symbol R
- D1, D2: footprint SOT-23 -> SOT-666; Farnell 1857788 -> 1295310
- IC6: footprint SOT563 -> SOT-563
- P10, P11, P12, P14, P15, P16, P17, P18, P19, P2, P20, P21, P22, P23, P25, P4, P5, P6, P7, P8, P9: footprint (none) -> TP
- Q1: footprint SOT-23 -> SOT-23-3
- SMA1: footprint SMA_JACK_END_LAUNCH -> SMA_JACK_END
Connections:
- net labels added: JNTRST, JTCK, JTDI, JTDO, JTMS
- net labels removed: STM_USB_DISC
- wire segments 520 -> 537
- no-connect marks 44 -> 40
Other:
- note added: "JTAG"
- note added: "STM USB\nD+ Pullup"
- note removed: "STM USB Disconnect"
- moved on the sheet: C10, C12, C16, C17, C8, C9, L1, R15, R20, R22, R7, R8

Commit message: respec jtag header for shrouded version
Parts:
- P26: Farnell 9689621 -> 1801396
Changed lines of the file:
@@
-EESchema Schematic File Version 2  date Sat 25 Feb 2012 20:38:11 GMT
+EESchema Schematic File Version 2  date Sat 25 Feb 2012 20:49:20 GMT
 LIBS:mosfet_n
 LIBS:npn
@@
 F 1 "CONN_10X2" V 10050 3500 50  0000 C CNN
 F 2 "HEADER_SMD_2X10WAY" H 10050 3600 60  0001 C CNN
-F 4 "9689621" H 10050 3600 60  0001 C CNN "Farnell"
+F 4 "1801396" H 10050 3600 60  0001 C CNN "Farnell"
 	1    10050 3600
 	1    0    0    -1

Commit message: respec cheaper and more available jtag header
Parts:
- P26: Farnell 1801396 -> 1428504
Changed lines of the file:
@@
-EESchema Schematic File Version 2  date Sat 25 Feb 2012 20:49:20 GMT
+EESchema Schematic File Version 2  date Sat 25 Feb 2012 20:53:19 GMT
 LIBS:mosfet_n
 LIBS:npn
@@
 F 1 "CONN_10X2" V 10050 3500 50  0000 C CNN
 F 2 "HEADER_SMD_2X10WAY" H 10050 3600 60  0001 C CNN
-F 4 "1801396" H 10050 3600 60  0001 C CNN "Farnell"
+F 4 "1428504" H 10050 3600 60  0001 C CNN "Farnell"
 	1    10050 3600
 	1    0    0    -1

Commit message: jtag header done, ready to rock and roll
Other:
- note added: "STM USB D+ Pullup\n(only required for\nSTM32F1x)"
- note removed: "STM USB\nD+ Pullup"
Changed lines of the file:
@@
-EESchema Schematic File Version 2  date Sat 25 Feb 2012 20:53:19 GMT
+EESchema Schematic File Version 2  date Sun 26 Feb 2012 00:09:08 GMT
 LIBS:mosfet_n
 LIBS:npn
@@
 Sheet 1 1
 Title "Wombat Flight Computer"
-Date "25 feb 2012"
+Date "26 feb 2012"
 Rev "1"
 Comp "CU Spaceflight"
@@
 Text Notes 1000 5800 0    60   ~ 0
 STM USB\nDetect
-Text Notes 3950 7550 0    60   ~ 0
-STM USB\nD+ Pullup
+Text Notes 3800 7550 0    60   ~ 0
+STM USB D+ Pullup\n(only required for\nSTM32F1x)
 Text Notes 10250 1050 0    60   ~ 0
 MAIN 3v3 SMPS

Commit message: move to 2x5 jtag header. all parts placed.
Parts:
- removed P26: CONN_10X2, HEADER_SMD_2X10WAY, symbol CONN_10X2
- added P26: CONN_5X2, HEADER_SMD_2X5WAY, symbol CONN_5X2
Connections:
- net labels removed: JNTRST
- wire segments 537 -> 540
- no-connect marks 40 -> 38
Other:
- note added: "JTAG/SWD"
- note removed: "JTAG"
- moved on the sheet: C34

Commit message: add micro sd card and begin the routing
Parts:
- added C50: 100n, SM0402, symbol C
- added R12: 22k, SM0402, symbol R
- added R18: 10k, SM0402, symbol R
- added U3: MICROSD, MICROSD, symbol MICROSD
Connections:
- net labels added: SDIO_CLK, SDIO_CMD, SDIO_D0, SD_CD
- wire segments 540 -> 572
- no-connect marks 38 -> 35
Other:
- moved on the sheet: R15, R20

Commit message: ONE LAST TRACE, ONE TRACE MORE
Connections:
- wire segments 572 -> 570
